File: PCB/RFUSBtoDB15Adapter.brd (EAGLE design)
At the start: 40.4 x 56.1 mm, 22 parts, among them IC1 S-816A40AMC-BAPT2U, J1 0, J2 AVR_SPI_PROG_3X2NS, Q2 2SA1213-Y(TE12L,F)

Commit message: New PCB and Schematics
PCB/Schematics REV 1.2
Parts:
- moved LED 1.91 mm to (33.1, 27.3)
- moved J2 1.08 mm to (38.2, 32.6)
Connections:
- net 5VREG: no longer J1.2, J2.2
- net 5VSG: now also J1.2, J2.2
Routing:
- net 5VSG: track 45.4 -> 129.9 mm, vias 4 -> 12
- net 5VREG: track 150.0 -> 129.9 mm
- net LED: track 21.8 -> 23.7 mm
- net LEDREG: track 14.0 -> 16.0 mm
- net START: track 65.3 -> 66.0 mm
- net MOSI: track 17.9 -> 18.5 mm
- net MISO: track 6.64 -> 7.17 mm
Other:
- board text added: "RST"
- board text added: "Reset Memory"
- board text added: "USB2DB15 Adapter for Supergun/Neogeo 1.2 by Raph_friend"
- board text removed: "RESET"
- board text removed: "USB2DB15 Adapter for Supergun/Neogeo 1.1 by Raph_friend"
