File: PCB/RFUSBtoDB15Adapter.sch (EAGLE design)
At the start: 21 parts, among them IC1 S-816A40AMC-BAPT2U, J1 0, J2 AVR_SPI_PROG_3X2NS, Q2 2SA1213-Y(TE12L,F)

Commit message: New PCB and Schematics
PCB/Schematics REV 1.2
Connections:
- net 5VREG: no longer J1.2, J2.2
- net 5VSG: now also J1.2, J2.2
Changed lines of the file:
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@@
 <?xml version="1.0" encoding="utf-8"?>
 <!DOCTYPE eagle SYSTEM "eagle.dtd">
-<eagle version="9.5.1">
+<eagle version="9.6.2">
 <drawing>
 <settings>
@@
 <part name="FRAME1" library="SparkFun-Aesthetics" library_urn="urn:adsk.eagle:library:507" deviceset="FRAME-A4L" device="">
 <attribute name="CNAME" value="USB2DB15 adapter for Supergun/Neogeo"/>
-<attribute name="CREVISION" value="1.1"/>
+<attribute name="CREVISION" value="1.2"/>
 <attribute name="DESIGNER" value="Design: Raph_friend"/>
 </part>
@@
 <label x="45.72" y="81.28" size="1.778" layer="95"/>
 </segment>
+<segment>
+<pinref part="J1" gate="G$1" pin="2"/>
+<wire x1="-137.16" y1="-40.64" x2="-147.32" y2="-40.64" width="0.1524" layer="91"/>
+<label x="-147.066" y="-40.64" size="1.778" layer="95" rot="R180"/>
+</segment>
+<segment>
+<pinref part="J2" gate="G$1" pin="2"/>
+<wire x1="-96.52" y1="-40.64" x2="-88.9" y2="-40.64" width="0.1524" layer="91"/>
+<label x="-93.98" y="-40.64" size="1.778" layer="95"/>
+</segment>
 </net>
 <net name="DTR" class="0">
@@
 </segment>
 <segment>
-<pinref part="J1" gate="G$1" pin="2"/>
-<wire x1="-137.16" y1="-40.64" x2="-147.32" y2="-40.64" width="0.1524" layer="91"/>
-<label x="-147.066" y="-40.64" size="1.778" layer="95" rot="R180"/>
-</segment>
-<segment>
-<pinref part="J2" gate="G$1" pin="2"/>
-<wire x1="-96.52" y1="-40.64" x2="-88.9" y2="-40.64" width="0.1524" layer="91"/>
-<label x="-93.98" y="-40.64" size="1.778" layer="95"/>
-</segment>
-<segment>
